Commit message: Spider man test 1

File: robots/go1_description/xacro/const.xacro (robot description, xacro)
@@ -53,13 +53,13 @@
     <xacro:property name="hip_position_min" value="-0.863"/>
     <xacro:property name="hip_velocity_max" value="30.1"/>
-    <xacro:property name="hip_torque_max" value="23.7"/>
+    <xacro:property name="hip_torque_max" value="100.0"/>
     <xacro:property name="thigh_position_max" value="4.501"/>
     <xacro:property name="thigh_position_min" value="-0.686"/>
     <xacro:property name="thigh_velocity_max" value="30.1"/>
-    <xacro:property name="thigh_torque_max" value="23.7"/>
+    <xacro:property name="thigh_torque_max" value="100.0"/>
     <xacro:property name="calf_position_max" value="-0.888"/>
     <xacro:property name="calf_position_min" value="-2.818"/>
     <xacro:property name="calf_velocity_max" value="20.06"/>
-    <xacro:property name="calf_torque_max" value="35.55"/>
+    <xacro:property name="calf_torque_max" value="100.0"/>
     <!-- dynamics inertial value        total 12.84kg -->
     <!-- trunk -->

Commit message: Slight tuning

File: robots/go1_description/xacro/const.xacro (robot description, xacro)
@@ -53,13 +53,13 @@
     <xacro:property name="hip_position_min" value="-0.863"/>
     <xacro:property name="hip_velocity_max" value="30.1"/>
-    <xacro:property name="hip_torque_max" value="100.0"/>
+    <xacro:property name="hip_torque_max" value="23.7"/>
     <xacro:property name="thigh_position_max" value="4.501"/>
     <xacro:property name="thigh_position_min" value="-0.686"/>
     <xacro:property name="thigh_velocity_max" value="30.1"/>
-    <xacro:property name="thigh_torque_max" value="100.0"/>
+    <xacro:property name="thigh_torque_max" value="23.7"/>
     <xacro:property name="calf_position_max" value="-0.888"/>
     <xacro:property name="calf_position_min" value="-2.818"/>
     <xacro:property name="calf_velocity_max" value="20.06"/>
-    <xacro:property name="calf_torque_max" value="100.0"/>
+    <xacro:property name="calf_torque_max" value="23.7"/>
     <!-- dynamics inertial value        total 12.84kg -->
     <!-- trunk -->

File: robots/go1_description/xacro/gazebo.xacro (robot description, xacro)
@@ -285,6 +285,6 @@
     </gazebo>
     <gazebo reference="FL_foot">
-        <mu1>0.6</mu1>
-        <mu2>0.6</mu2>
+        <mu1>1.0</mu1>
+        <mu2>1.0</mu2>
         <self_collide>1</self_collide>
         <material>Gazebo/DarkGrey</material>
@@ -312,6 +312,6 @@
     </gazebo>
     <gazebo reference="FR_foot">
-        <mu1>0.6</mu1>
-        <mu2>0.6</mu2>
+        <mu1>1.0</mu1>
+        <mu2>1.0</mu2>
         <self_collide>1</self_collide>
         <material>Gazebo/DarkGrey</material>
@@ -339,6 +339,6 @@
     </gazebo>
     <gazebo reference="RL_foot">
-        <mu1>0.6</mu1>
-        <mu2>0.6</mu2>
+        <mu1>1.0</mu1>
+        <mu2>1.0</mu2>
         <self_collide>1</self_collide>
         <material>Gazebo/DarkGrey</material>
@@ -366,6 +366,6 @@
     </gazebo>
     <gazebo reference="RR_foot">
-        <mu1>0.6</mu1>
-        <mu2>0.6</mu2>
+        <mu1>1.0</mu1>
+        <mu2>1.0</mu2>
         <self_collide>1</self_collide>
         <material>Gazebo/DarkGrey</material>

Commit message: WIP

File: robots/go1_description/xacro/const.xacro (robot description, xacro)
@@ -53,13 +53,13 @@
     <xacro:property name="hip_position_min" value="-0.863"/>
     <xacro:property name="hip_velocity_max" value="30.1"/>
-    <xacro:property name="hip_torque_max" value="23.7"/>
+    <xacro:property name="hip_torque_max" value="100.0"/>
     <xacro:property name="thigh_position_max" value="4.501"/>
     <xacro:property name="thigh_position_min" value="-0.686"/>
     <xacro:property name="thigh_velocity_max" value="30.1"/>
-    <xacro:property name="thigh_torque_max" value="23.7"/>
+    <xacro:property name="thigh_torque_max" value="100.0"/>
     <xacro:property name="calf_position_max" value="-0.888"/>
     <xacro:property name="calf_position_min" value="-2.818"/>
     <xacro:property name="calf_velocity_max" value="20.06"/>
-    <xacro:property name="calf_torque_max" value="23.7"/>
+    <xacro:property name="calf_torque_max" value="100.0"/>
     <!-- dynamics inertial value        total 12.84kg -->
     <!-- trunk -->

File: robots/go1_description/xacro/gazebo.xacro (robot description, xacro)
@@ -280,11 +280,11 @@
     </gazebo>
     <gazebo reference="FL_calf">
-        <mu1>0.2</mu1>
-        <mu2>0.2</mu2>
+        <mu1>Inf</mu1>
+        <mu2>Inf</mu2>
         <self_collide>1</self_collide>
     </gazebo>
     <gazebo reference="FL_foot">
-        <mu1>1.0</mu1>
-        <mu2>1.0</mu2>
+        <mu1>0.6</mu1>
+        <mu2>0.6</mu2>
         <self_collide>1</self_collide>
         <material>Gazebo/DarkGrey</material>
@@ -307,11 +307,11 @@
     </gazebo>
     <gazebo reference="FR_calf">
-        <mu1>0.2</mu1>
-        <mu2>0.2</mu2>
+        <mu1>Inf</mu1>
+        <mu2>Inf</mu2>
         <self_collide>1</self_collide>
     </gazebo>
     <gazebo reference="FR_foot">
-        <mu1>1.0</mu1>
-        <mu2>1.0</mu2>
+        <mu1>0.6</mu1>
+        <mu2>0.6</mu2>
         <self_collide>1</self_collide>
         <material>Gazebo/DarkGrey</material>
@@ -334,11 +334,11 @@
     </gazebo>
     <gazebo reference="RL_calf">
-        <mu1>0.2</mu1>
-        <mu2>0.2</mu2>
+        <mu1>Inf</mu1>
+        <mu2>Inf</mu2>
         <self_collide>1</self_collide>
     </gazebo>
     <gazebo reference="RL_foot">
-        <mu1>1.0</mu1>
-        <mu2>1.0</mu2>
+        <mu1>0.6</mu1>
+        <mu2>0.6</mu2>
         <self_collide>1</self_collide>
         <material>Gazebo/DarkGrey</material>
@@ -361,11 +361,11 @@
     </gazebo>
     <gazebo reference="RR_calf">
-        <mu1>0.2</mu1>
-        <mu2>0.2</mu2>
+        <mu1>Inf</mu1>
+        <mu2>Inf</mu2>
         <self_collide>1</self_collide>
     </gazebo>
     <gazebo reference="RR_foot">
-        <mu1>1.0</mu1>
-        <mu2>1.0</mu2>
+        <mu1>0.6</mu1>
+        <mu2>0.6</mu2>
         <self_collide>1</self_collide>
         <material>Gazebo/DarkGrey</material>

Commit message: Adjustment

File: robots/go1_description/xacro/const.xacro (robot description, xacro)
@@ -5,18 +5,18 @@
     <xacro:property name="stick_mass" value="0.00001"/>
     <!-- simplified collision value -->
-    <xacro:property name="trunk_width" value="0.0935"/>
-    <xacro:property name="trunk_length" value="0.3762"/>
-    <xacro:property name="trunk_height" value="0.114"/>
-    <xacro:property name="hip_radius" value="0.046"/>
-    <xacro:property name="hip_length" value="0.04"/>
-    <xacro:property name="thigh_shoulder_radius" value="0.041"/>
-    <xacro:property name="thigh_shoulder_length" value="0.032"/>
-    <xacro:property name="thigh_width" value="0.0245"/>
-    <xacro:property name="thigh_height" value="0.034"/>
-    <xacro:property name="calf_width" value="0.016"/>
-    <xacro:property name="calf_height" value="0.016"/>
+    <xacro:property name="trunk_width" value="0.01"/>
+    <xacro:property name="trunk_length" value="0.01"/>
+    <xacro:property name="trunk_height" value="0.01"/>
+    <xacro:property name="hip_radius" value="0.01"/>
+    <xacro:property name="hip_length" value="0.01"/>
+    <xacro:property name="thigh_shoulder_radius" value="0.01"/>
+    <xacro:property name="thigh_shoulder_length" value="0.01"/>
+    <xacro:property name="thigh_width" value="0.01"/>
+    <xacro:property name="thigh_height" value="0.01"/>
+    <xacro:property name="calf_width" value="0.01"/>
+    <xacro:property name="calf_height" value="0.01"/>
     <xacro:property name="foot_radius" value="0.02"/>
     <xacro:property name="stick_radius" value="0.01"/>
-    <xacro:property name="stick_length" value="0.2"/>
+    <xacro:property name="stick_length" value="0.01"/>
     <!-- kinematic value -->
     <xacro:property name="thigh_offset" value="0.08"/>
@@ -50,14 +50,14 @@
     <xacro:property name="damping" value="0.01"/>
     <xacro:property name="friction" value="0.2"/>
-    <xacro:property name="hip_position_max" value="0.863"/>
-    <xacro:property name="hip_position_min" value="-0.863"/>
+    <xacro:property name="hip_position_max" value="6.28"/>
+    <xacro:property name="hip_position_min" value="-6.28"/>
     <xacro:property name="hip_velocity_max" value="30.1"/>
     <xacro:property name="hip_torque_max" value="100.0"/>
-    <xacro:property name="thigh_position_max" value="4.501"/>
-    <xacro:property name="thigh_position_min" value="-0.686"/>
+    <xacro:property name="thigh_position_max" value="6.28"/>
+    <xacro:property name="thigh_position_min" value="-6.28"/>
     <xacro:property name="thigh_velocity_max" value="30.1"/>
     <xacro:property name="thigh_torque_max" value="100.0"/>
-    <xacro:property name="calf_position_max" value="-0.888"/>
-    <xacro:property name="calf_position_min" value="-2.818"/>
+    <xacro:property name="calf_position_max" value="6.28"/>
+    <xacro:property name="calf_position_min" value="-6.28"/>
     <xacro:property name="calf_velocity_max" value="20.06"/>
     <xacro:property name="calf_torque_max" value="100.0"/>
