Commit message: Update

File: robots/a1_rw_description/xacro/gazebo.xacro (robot description, xacro)
@@ -35,5 +35,5 @@
             <always_on>true</always_on>
             <update_rate>200</update_rate>
-            <bodyName>base</bodyName>
+            <bodyName>trunk</bodyName>
             <topicName>/torso_odom</topicName>
             <frameName>world</frameName>

File: robots/a1_rw_description/xacro/robot.xacro (robot description, xacro)
@@ -7,5 +7,4 @@
     <xacro:include filename="$(find a1_rw_description)/xacro/stairs.xacro"/>
     <xacro:include filename="$(find a1_rw_description)/xacro/gazebo.xacro"/>
-    <!-- <xacro:stairs stairs="15" xpos="0" ypos="0" zpos="0" /> -->
     <!-- Rollover Protection mode will add an additional stick on the top, use "true" or "false" to switch it. -->
     <xacro:property name="rolloverProtection" value="false"/>
@@ -40,10 +39,4 @@
             <material name="orange"/>
         </visual>
-        <collision>
-            <origin rpy="0 0 0" xyz="0 0 0"/>
-            <geometry>
-                <box size="${trunk_length} ${trunk_width} ${trunk_height}"/>
-            </geometry>
-        </collision>
         <inertial>
             <origin rpy="0 0 0" xyz="${trunk_com_x} ${trunk_com_y} ${trunk_com_z}"/>
@@ -55,33 +48,4 @@
         </inertial>
     </link>
-    <xacro:if value="${(rolloverProtection == 'true')}">
-        <joint name="stick_joint" type="fixed">
-            <parent link="trunk"/>
-            <child link="stick_link"/>
-            <origin rpy="0 0 0" xyz="${0.18} 0 ${stick_length/2.0+0.08}"/>
-        </joint>
-        <link name="stick_link">
-            <visual>
-                <geometry>
-                    <cylinder length="${stick_length}" radius="${stick_radius}"/>
-                </geometry>
-                <origin rpy="0 0 0" xyz="0 0 0"/>
-                <material name="white"/>
-            </visual>
-            <collision>
-                <geometry>
-                    <cylinder length="${stick_length}" radius="${stick_radius}"/>
-                </geometry>
-                <origin rpy="0 0 0" xyz="0 0 0"/>
-            </collision>
-            <inertial>
-                <mass value="${stick_mass}"/>
-                <inertia
-                    ixx="${stick_mass / 2.0 * (stick_radius*stick_radius)}" ixy="0.0" ixz="0.0"
-                    iyy="${stick_mass / 12.0 * (3*stick_radius*stick_radius + stick_length*stick_length)}" iyz="0.0"
-                    izz="${stick_mass / 12.0 * (3*stick_radius*stick_radius + stick_length*stick_length)}"/>
-            </inertial>
-        </link>
-    </xacro:if>
     <joint name="imu_joint" type="fixed">
         <parent link="trunk"/>
@@ -109,163 +73,83 @@
         </collision>
     </link>
-    <link
-    name="base_link">
-    <inertial>
-      <origin
-        xyz="0.0026038995042581 -0.0740490943270337 0.0694515969568454"
-        rpy="0 0 0" />
-      <mass
-        value="2.27585184177867" />
-      <inertia
-        ixx="0.00269192131058548"
-        ixy="-1.60048667500493E-06"
-        ixz="2.62534222384217E-07"
-        iyy="0.00322414588067439"
-        iyz="0.000180161400738552"
-        izz="0.00320797475119015" />
-    </inertial>
-    <visual>
-      <origin
-        xyz="0 0 0"
-        rpy="0 0 0" />
-      <geometry>
-        <mesh
-          filename="package://a1_rw_description/meshes/base_link.STL" />
-      </geometry>
-      <material
-        name="">
-        <color
-          rgba="0.847058823529412 0.847058823529412 0.847058823529412 1" />
-      </material>
-    </visual>
-    <collision>
-      <origin
-        xyz="0 0 0"
-        rpy="0 0 0" />
-      <geometry>
-        <mesh
-          filename="package://a1_rw_description/meshes/base_link.STL" />
-      </geometry>
-    </collision>
-  </link>
-  <joint
-    name="backpack_connection"
-    type="fixed">
-    <origin
-      xyz="0 0 0.055"
-      rpy="0 0 1.57079632679489" />
-    <parent
-      link="base" />
-    <child
-      link="base_link" />
-  </joint>
-  <link
-    name="rwx">
-    <inertial>
-      <origin
-        xyz="2.11694828333719E-11 4.47206311478959E-10 0.0346816748196828"
-        rpy="0 0 0" />
-      <mass
-        value="1.30351405536484" />
-      <inertia
-        ixx="0.00271165021972425"
-        ixy="1.62817777047674E-08"
-        ixz="-8.58134995976747E-12"
-        iyy="0.00271170564663939"
-        iyz="1.07399173903702E-11"
-        izz="0.00527518299832296" />
-    </inertial>
-    <visual>
-      <origin
-        xyz="0 0 0"
-        rpy="0 0 0" />
-      <geometry>
-        <mesh
-          filename="package://a1_rw_description/meshes/rwx.STL" />
-      </geometry>
-      <material
-        name="">
-        <color
-          rgba="0.752941176470588 0.752941176470588 0.752941176470588 1" />
-      </material>
-    </visual>
-    <collision>
-      <origin
-        xyz="0 0 0"
-        rpy="0 0 0" />
-      <geometry>
-        <mesh
-          filename="package://a1_rw_description/meshes/rwx.STL" />
-      </geometry>
-    </collision>
-  </link>
-  <joint
-    name="joint_rwx"
-    type="continuous">
-    <origin
-      xyz="0 -0.09729 0.0919999999999999"
-      rpy="-1.5707963267949 0 0" />
-    <parent
-      link="base_link" />
-    <child
-      link="rwx" />
-    <axis
-      xyz="0 0 1" />
-    <dynamics damping="0.0" friction="0."/>
-  </joint>
-  <link
-    name="rwy">
-    <inertial>
-      <origin
-        xyz="-2.54625994081104E-07 7.07442964209548E-08 0.0364184294382762"
-        rpy="0 0 0" />
-      <mass
-        value="1.12728695649087" />
-      <inertia
-        ixx="0.000962317962998777"
-        ixy="1.4679589412309E-08"
-        ixz="6.6087002464196E-11"
-        iyy="0.000962369623284224"
-        iyz="1.53941482098914E-11"
-        izz="0.00189043287041886" />
-    </inertial>
-    <visual>
-      <origin
-        xyz="0 0 0"
-        rpy="0 0 0" />
-      <geometry>
-        <mesh
-          filename="package://a1_rw_description/meshes/rwy.STL" />
-      </geometry>
-      <material
-        name="">
-        <color
-          rgba="0.752941176470588 0.752941176470588 0.752941176470588 1" />
-      </material>
-    </visual>
-    <collision>
-      <origin
-        xyz="0 0 0"
-        rpy="0 0 0" />
-      <geometry>
-        <mesh
-          filename="package://a1_rw_description/meshes/rwy.STL" />
-      </geometry>
-    </collision>
-  </link>
-  <joint
-    name="joint_rwy"
-    type="continuous">
-    <origin
-      xyz="0.0324749999999997 0.0569999999999978 0.0920000000000013"
-      rpy="1.57079632679489 -0.651399930466687 -1.57079632679489" />
-    <parent
-      link="base_link" />
-    <child
-      link="rwy" />
-    <axis
-      xyz="0 0 -1" />
-    <dynamics damping="0.0" friction="0."/>
-  </joint>
+    <link name="base_link">
+        <inertial>
+            <origin xyz="0.0026038995042581 -0.0740490943270337 0.0694515969568454" rpy="0 0 0"/>
+            <mass value="2.27585184177867"/>
+            <inertia ixx="0.00269192131058548" ixy="-1.60048667500493E-06" ixz="2.62534222384217E-07" iyy="0.00322414588067439" iyz="0.000180161400738552" izz="0.00320797475119015"/>
+        </inertial>
+        <visual>
+            <origin xyz="0 0 0" rpy="0 0 0"/>
+            <geometry>
+                <mesh filename="package://a1_rw_description/meshes/base_link.STL"/>
+            </geometry>
+            <material name="">
+                <color rgba="0.847058823529412 0.847058823529412 0.847058823529412 1"/>
+            </material>
+        </visual>
+    </link>
+    <joint name="backpack_connection" type="fixed">
+        <origin xyz="0 0 0.055" rpy="0 0 1.57079632679489"/>
+        <parent link="trunk"/>
+        <child link="base_link"/>
+    </joint>
+    <link name="rwx">
+        <inertial>
+            <origin xyz="2.11694828333719E-11 4.47206311478959E-10 0.0346816748196828" rpy="0 0 0"/>
+            <mass value="1.30351405536484"/>
+            <inertia ixx="0.00271165021972425" ixy="1.62817777047674E-08" ixz="-8.58134995976747E-12" iyy="0.00271170564663939" iyz="1.07399173903702E-11" izz="0.00527518299832296"/>
+        </inertial>
+        <visual>
+            <origin xyz="0 0 0" rpy="0 0 0"/>
+            <geometry>
+                <mesh filename="package://a1_rw_description/meshes/rwx.STL"/>
+            </geometry>
+            <material name="">
+                <color rgba="0.752941176470588 0.752941176470588 0.752941176470588 1"/>
+            </material>
+        </visual>
+        <collision>
+            <origin xyz="0 0 0" rpy="0 0 0"/>
+            <geometry>
+                <mesh filename="package://a1_rw_description/meshes/rwx.STL"/>
+            </geometry>
+        </collision>
+    </link>
+    <joint name="joint_rwx" type="continuous">
+        <origin xyz="0 -0.09729 0.0919999999999999" rpy="-1.5707963267949 0 0"/>
+        <parent link="base_link"/>
+        <child link="rwx"/>
+        <axis xyz="0 0 1"/>
+        <dynamics damping="0.0" friction="0."/>
+    </joint>
+    <link name="rwy">
+        <inertial>
+            <origin xyz="-2.54625994081104E-07 7.07442964209548E-08 0.0364184294382762" rpy="0 0 0"/>
+            <mass value="1.12728695649087"/>
+            <inertia ixx="0.000962317962998777" ixy="1.4679589412309E-08" ixz="6.6087002464196E-11" iyy="0.000962369623284224" iyz="1.53941482098914E-11" izz="0.00189043287041886"/>
+        </inertial>
+        <visual>
+            <origin xyz="0 0 0" rpy="0 0 0"/>
+            <geometry>
+                <mesh filename="package://a1_rw_description/meshes/rwy.STL"/>
+            </geometry>
+            <material name="">
+                <color rgba="0.752941176470588 0.752941176470588 0.752941176470588 1"/>
+            </material>
+        </visual>
+        <collision>
+            <origin xyz="0 0 0" rpy="0 0 0"/>
+            <geometry>
+                <mesh filename="package://a1_rw_description/meshes/rwy.STL"/>
+            </geometry>
+        </collision>
+    </link>
+    <joint name="joint_rwy" type="continuous">
+        <origin xyz="0.0324749999999997 0.0569999999999978 0.0920000000000013" rpy="1.57079632679489 -0.651399930466687 -1.57079632679489"/>
+        <parent link="base_link"/>
+        <child link="rwy"/>
+        <axis xyz="0 0 -1"/>
+        <dynamics damping="0.0" friction="0."/>
+    </joint>
     <xacro:leg name="FR" mirror="-1" mirror_dae="False" front_hind="1" front_hind_dae="True">
         <origin rpy="0 0 0" xyz="${leg_offset_x} ${-leg_offset_y} 0"/>
@@ -280,4 +164,3 @@
         <origin rpy="0 0 0" xyz="${-leg_offset_x} ${leg_offset_y} 0"/>
     </xacro:leg>
-    <!-- <xacro:stairs stairs="15" xpos="0" ypos="2.0" zpos="0" /> -->
 </robot>

File: robots/a1_rw_description/xacro/transmission.xacro (robot description, xacro)
@@ -32,24 +32,24 @@
             </actuator>
         </transmission>
+        <transmission name="wheel_x_trans">
+                <type>transmission_interface/SimpleTransmission</type>
+                <joint name="joint_rwx">
+                    <hardwareInterface>hardware_interface/EffortJointInterface</hardwareInterface>
+                </joint>
+                <actuator name="wheel_x_motor">
+                    <hardwareInterface>hardware_interface/EffortJointInterface</hardwareInterface>
+                    <mechanicalReduction>1</mechanicalReduction>
+                </actuator>
+        </transmission>
+        <transmission name="wheel_y_trans">
+                <type>transmission_interface/SimpleTransmission</type>
+                <joint name="joint_rwy">
+                    <hardwareInterface>hardware_interface/EffortJointInterface</hardwareInterface>
+                </joint>
+                <actuator name="wheel_y_motor">
+                    <hardwareInterface>hardware_interface/EffortJointInterface</hardwareInterface>
+                    <mechanicalReduction>1</mechanicalReduction>
+                </actuator>
+        </transmission>
     </xacro:macro>
-    <transmission name="wheel_x_trans">
-            <type>transmission_interface/SimpleTransmission</type>
-            <joint name="joint_rwx">
-                <hardwareInterface>hardware_interface/EffortJointInterface</hardwareInterface>
-            </joint>
-            <actuator name="wheel_x_motor">
-                <hardwareInterface>hardware_interface/EffortJointInterface</hardwareInterface>
-                <mechanicalReduction>1</mechanicalReduction>
-            </actuator>
-    </transmission>
-    <transmission name="wheel_y_trans">
-            <type>transmission_interface/SimpleTransmission</type>
-            <joint name="joint_rwy">
-                <hardwareInterface>hardware_interface/EffortJointInterface</hardwareInterface>
-            </joint>
-            <actuator name="wheel_y_motor">
-                <hardwareInterface>hardware_interface/EffortJointInterface</hardwareInterface>
-                <mechanicalReduction>1</mechanicalReduction>
-            </actuator>
-    </transmission>
 </robot>
